Commit message: Robotic arm with 5 DOF v1.1

File: urdf/seven_dof_arm.urdf (robot description, URDF)
Before this commit: robot arm_model, 7 links, 6 joints
Links:
- added link finger_link1, mass 1; collision box size=0.08 0.01 0.01; visual box size=0.08 0.01 0.01
- added link finger_link2, mass 1; collision box size=0.08 0.01 0.01; visual box size=0.08 0.01 0.01
- added link gripper_roll_link, mass 1; collision cylinder length=0.02 radius=0.04; visual cylinder length=0.02 radius=0.04
- added link wrist_pitch_link, mass 1; collision box size=0.06 0.04 0.04; visual box size=0.06 0.04 0.04
Joints:
- added joint finger_joint1: type prismatic, parent gripper_roll_link, child finger_link1, origin xyz=0.0 0 0, axis 0 1 0, limit lower=0 upper=0.03 effort=100 velocity=1.0
- added joint finger_joint2: type prismatic, parent gripper_roll_link, child finger_link2, origin xyz=0.0 0 0, axis 0 1 0, limit lower=-0.03 upper=0 effort=1 velocity=1.0
- added joint gripper_roll_joint: type revolute, parent wrist_pitch_link, child gripper_roll_link, origin xyz=0 0 0.080 rpy=4.712385 -1.570795 0, axis 1 0 0, limit lower=-3.14 upper=3.14 effort=300 velocity=1
- added joint wrist_pitch_joint: type revolute, parent wrist_roll_link, child wrist_pitch_link, origin xyz=0.0 0.0 0.0001 rpy=0 1.570795 0, axis 1 0 0, limit lower=-1.5953400194 upper=1.98394848567 effort=300 velocity=1
